Commit message: working g500 with arm

File: src/underwater/catkin_ws/src/g500arm5_description/urdf/g500arm5.urdf (robot description, URDF)
Before this commit: robot girona500, 1 links, 0 joints
Links:
- added link part0, mass 10; collision cylinder length=0.6 radius=0.2; visual mesh filename=package://g500arm5_description/meshes/ARM5E/ARM5E_part0.dae
- added link part1, mass 10; collision cylinder length=0.6 radius=0.2; visual mesh filename=package://g500arm5_description/meshes/ARM5E/ARM5E_part1.dae
- added link part2, mass 10; collision cylinder length=0.6 radius=0.2; visual mesh filename=package://g500arm5_description/meshes/ARM5E/ARM5E_part2.dae
- added link part3, mass 10; collision cylinder length=0.6 radius=0.2; visual mesh filename=package://g500arm5_description/meshes/ARM5E/ARM5E_part3.stl
- added link part4_base, mass 10; collision cylinder length=0.6 radius=0.2; visual mesh filename=package://g500arm5_description/meshes/ARM5E/ARM5E_part4_bas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
- added link part4_jaw1, mass 10; collision cylinder length=0.6 radius=0.2; visual mesh filename=package://g500arm5_description/meshes/ARM5E/ARM5E_part4_jaw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
- added link part4_jaw2, mass 10; collision cylinder length=0.6 radius=0.2; visual mesh filename=package://g500arm5_description/meshes/ARM5E/ARM5E_part4_jaw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
Joints:
- added joint baselink_to_part0: type fixed, parent base_link, child part0, origin xyz=-0.2 0 -.2 rpy=0 0 0
- added joint part0_to_part1: type continuous, parent part0, child part1, origin xyz=0 0 0 rpy=0 0 0, axis 0 0 -1
- added joint part1_to_part2: type continuous, parent part1, child part2, origin xyz=0.077 0 -0.130 rpy=0 0.209 0, axis 0 1 0
- added joint part2_to_part3: type continuous, parent part2, child part3, origin xyz=0.44278 0 0 rpy= 0 0.262 0 , axis 0 1 0
- added joint part3_to_part4_base: type continuous, parent part3, child part4_base, origin xyz=0.320 0 0.077  rpy=0 0 0, axis 1 0 0
- added joint part4_to_part4_jaw1: type continuous, parent part4_base, child part4_jaw1, origin xyz=0.07 0 0.04 rpy=0 0 0, axis 0 -1 0
- added joint part4_to_part4_jaw2: type continuous, parent part4_base, child part4_jaw2, origin xyz=0.07 0 -0.04 rpy=0 0 0, axis 0 1 0, mimic joint=part4_to_part4_jaw1 multiplier=1 offset=0
