Commit message: g500 in gazebo without freaking out

File: src/underwater/catkin_ws/src/g500arm5_description/urdf/g500arm5.xacro (robot description, xacro)
@@ -1,28 +1,8 @@
 <?xml version="1.0"?>
-<robot name="girona500">
-  <gazebo reference="base_link">
-    <gravity>0</gravity>
-  </gazebo>
-  <gazebo reference="part0">
-    <gravity>0</gravity>
-  </gazebo>
-  <gazebo reference="part1">
-    <gravity>0</gravity>
-  </gazebo>
-  <gazebo reference="part2">
-    <gravity>0</gravity>
-  </gazebo>
-  <gazebo reference="part3">
-    <gravity>0</gravity>
-  </gazebo>
-  <gazebo reference="part4_base">
-    <gravity>0</gravity>
-  </gazebo>
-  <gazebo reference="part4_jaw1">
-    <gravity>0</gravity>
-  </gazebo>
-  <gazebo reference="part4_jaw2">
-    <gravity>0</gravity>
-  </gazebo>
+<robot name="girona500" xmlns:xacro="http://www.ros.org/wiki/xacro">
+  <!-- Import all Gazebo-customization elements, including Gazebo colors -->
+  <xacro:include filename="$(find g500arm5_description)/urdf/g500arm5.gazebo" />
+  <!-- Import Rviz colors -->
+  <xacro:include filename="$(find g500arm5_description)/urdf/materials.xacro" />
   <link name="base_link">
     <visual>
@@ -38,6 +18,8 @@
     </collision>
     <inertial>
-      <mass value="10"/>
-      <inertia ixx="0.4" ixy="0.0" ixz="0.0" iyy="0.4" iyz="0.0" izz="0.2"/>
+      <mass value="98"/>
+      <inertia ixx="8.0" ixy="0.0" ixz="0.0"
+                         iyy="8.0" iyz="0.0"
+                                   izz="8.0"/>
     </inertial>
   </link>
@@ -51,10 +33,12 @@
     <collision>
       <geometry>
-        <cylinder length="0.6" radius="0.2"/>
-      </geometry>
-    </collision>
-    <inertial>
-      <mass value="10"/>
-      <inertia ixx="0.4" ixy="0.0" ixz="0.0" iyy="0.4" iyz="0.0" izz="0.2"/>
+        <box size="0.02 0.02 0.02" />
+      </geometry>
+    </collision>
+    <inertial>
+      <mass value="0.01"/>
+      <inertia ixx="6.667e-7" ixy="0.0"       ixz="0.0"
+                              iyy="6.667e-7"  iyz="0.0"
+                                              izz="6.667e-7" />
     </inertial>
   </link>
@@ -73,10 +57,12 @@
     <collision>
       <geometry>
-        <cylinder length="0.6" radius="0.2"/>
-      </geometry>
-    </collision>
-    <inertial>
-      <mass value="10"/>
-      <inertia ixx="0.4" ixy="0.0" ixz="0.0" iyy="0.4" iyz="0.0" izz="0.2"/>
+        <box size="0.02 0.02 0.02" />
+      </geometry>
+    </collision>
+    <inertial>
+      <mass value="0.01"/>
+      <inertia ixx="6.667e-7" ixy="0.0"       ixz="0.0"
+                              iyy="6.667e-7"  iyz="0.0"
+                                              izz="6.667e-7" />
     </inertial>
   </link>
@@ -96,10 +82,12 @@
     <collision>
       <geometry>
-        <cylinder length="0.6" radius="0.2"/>
-      </geometry>
-    </collision>
-    <inertial>
-      <mass value="10"/>
-      <inertia ixx="0.4" ixy="0.0" ixz="0.0" iyy="0.4" iyz="0.0" izz="0.2"/>
+        <box size="0.02 0.02 0.02" />
+      </geometry>
+    </collision>
+    <inertial>
+      <mass value="0.01"/>
+      <inertia ixx="6.667e-7" ixy="0.0"       ixz="0.0"
+                              iyy="6.667e-7"  iyz="0.0"
+                                              izz="6.667e-7" />
     </inertial>
   </link>
@@ -119,10 +107,12 @@
     <collision>
       <geometry>
-        <cylinder length="0.6" radius="0.2"/>
-      </geometry>
-    </collision>
-    <inertial>
-      <mass value="10"/>
-      <inertia ixx="0.4" ixy="0.0" ixz="0.0" iyy="0.4" iyz="0.0" izz="0.2"/>
+        <box size="0.02 0.02 0.02" />
+      </geometry>
+    </collision>
+    <inertial>
+      <mass value="0.01"/>
+      <inertia ixx="6.667e-7" ixy="0.0"      ixz="0.0"
+                              iyy="6.667e-7" iyz="0.0"
+                                             izz="6.667e-7" />
     </inertial>
   </link>
@@ -133,5 +123,5 @@
     <origin rpy=" 0 0.262 0 " xyz="0.44278 0 0"/>
   </joint>
-  <link name="part4_base">
+    <link name="part4_base">
     <visual>
       <origin rpy="0 0 0" xyz="0 0 0"/>
@@ -142,10 +132,12 @@
     <collision>
       <geometry>
-        <cylinder length="0.6" radius="0.2"/>
-      </geometry>
-    </collision>
-    <inertial>
-      <mass value="10"/>
-      <inertia ixx="0.4" ixy="0.0" ixz="0.0" iyy="0.4" iyz="0.0" izz="0.2"/>
+        <box size="0.02 0.02 0.02" />
+      </geometry>
+    </collision>
+    <inertial>
+      <mass value="0.01"/>
+      <inertia ixx="6.667e-7" ixy="0.0"       ixz="0.0"
+                              iyy="6.667e-7"  iyz="0.0"
+                                              izz="6.667e-7" />
     </inertial>
   </link>
@@ -165,10 +157,12 @@
     <collision>
       <geometry>
-        <cylinder length="0.6" radius="0.2"/>
-      </geometry>
-    </collision>
-    <inertial>
-      <mass value="10"/>
-      <inertia ixx="0.4" ixy="0.0" ixz="0.0" iyy="0.4" iyz="0.0" izz="0.2"/>
+        <box size="0.02 0.02 0.02" />
+      </geometry>
+    </collision>
+    <inertial>
+      <mass value="0.01"/>
+      <inertia ixx="6.667e-7" ixy="0.0"       ixz="0.0"
+                              iyy="6.667e-7"  iyz="0.0"
+                                              izz="6.667e-7" />
     </inertial>
   </link>
@@ -188,10 +182,12 @@
     <collision>
       <geometry>
-        <cylinder length="0.6" radius="0.2"/>
-      </geometry>
-    </collision>
-    <inertial>
-      <mass value="10"/>
-      <inertia ixx="0.4" ixy="0.0" ixz="0.0" iyy="0.4" iyz="0.0" izz="0.2"/>
+        <box size="0.02 0.02 0.02" />
+      </geometry>
+    </collision>
+    <inertial>
+      <mass value="0.01"/>
+      <inertia ixx="6.667e-7" ixy="0.0"       ixz="0.0"
+                              iyy="6.667e-7"  iyz="0.0"
+                                              izz="6.667e-7" />
     </inertial>
   </link>

Commit message: working velocity control from ros

File: src/underwater/catkin_ws/src/g500arm5_description/urdf/g500arm5.xacro (robot description, xacro)
@@ -7,5 +7,5 @@
   <link name="base_link">
     <visual>
-      <origin rpy="1.57 0 0" xyz="0 0 0"/>
+      <origin rpy="1.57 0 3.14156" xyz="0 0 0"/>
       <geometry>
         <mesh filename="package://g500arm5_description/meshes/GIRONA500/g500.dae"/>
@@ -72,4 +72,5 @@
     <axis xyz="0 0 -1"/>
     <origin rpy="0 0 0" xyz="0 0 0"/>
+    <dynamics damping="0.5"/>
   </joint>
   <link name="part2">
@@ -97,4 +98,5 @@
     <axis xyz="0 1 0"/>
     <origin rpy="0 0.209 0" xyz="0.077 0 -0.130"/>
+    <dynamics damping="0.5"/>
   </joint>
   <link name="part3">
@@ -122,4 +124,5 @@
     <axis xyz="0 1 0"/>
     <origin rpy=" 0 0.262 0 " xyz="0.44278 0 0"/>
+    <dynamics damping="0.5"/>
   </joint>
     <link name="part4_base">
@@ -147,4 +150,5 @@
     <axis xyz="1 0 0"/>
     <origin rpy="0 0 0" xyz="0.320 0 0.077 "/>
+    <dynamics damping="0.5"/>
   </joint>
   <link name="part4_jaw1">
@@ -172,4 +176,5 @@
     <axis xyz="0 -1 0"/>
     <origin rpy="0 0 0" xyz="0.07 0 0.04"/>
+    <dynamics damping="0.5"/>
   </joint>
   <link name="part4_jaw2">

Commit message: added setworldpose to velcmd

File: src/underwater/catkin_ws/src/g500arm5_description/urdf/g500arm5.xacro (robot description, xacro)
@@ -7,5 +7,5 @@
   <link name="base_link">
     <visual>
-      <origin rpy="1.57 0 3.14156" xyz="0 0 0"/>
+      <origin rpy="1.57079 0 0" xyz="0 0 0"/>
       <geometry>
         <mesh filename="package://g500arm5_description/meshes/GIRONA500/g500.dae"/>

Commit message: verified dynamics, fixing bounds on arm

File: src/underwater/catkin_ws/src/g500arm5_description/urdf/g500arm5.xacro (robot description, xacro)
@@ -7,5 +7,5 @@
   <link name="base_link">
     <visual>
-      <origin rpy="1.57079 0 0" xyz="0 0 0"/>
+      <origin rpy="1.57079 0 3.1416" xyz="0 0 0"/>
       <geometry>
         <mesh filename="package://g500arm5_description/meshes/GIRONA500/g500.dae"/>
@@ -14,5 +14,5 @@
     <collision>
       <geometry>
-        <cylinder length="0.6" radius="0.2"/>
+        <cylinder length="1.5" radius="0.35"/>
       </geometry>
     </collision>
@@ -33,5 +33,5 @@
     <collision>
       <geometry>
-        <box size="0.02 0.02 0.02" />
+        <box size="0.35 0.13 0.10" />
       </geometry>
     </collision>
@@ -57,5 +57,5 @@
     <collision>
       <geometry>
-        <box size="0.02 0.02 0.02" />
+        <box size="0.10 0.16 0.15" />
       </geometry>
     </collision>
@@ -71,5 +71,5 @@
     <child link="part1"/>
     <axis xyz="0 0 -1"/>
-    <origin rpy="0 0 0" xyz="0 0 0"/>
+    <origin rpy="0 0 1.57" xyz="0 0 0"/>
     <dynamics damping="0.5"/>
   </joint>
@@ -83,5 +83,5 @@
     <collision>
       <geometry>
-        <box size="0.02 0.02 0.02" />
+        <box size="0.60 0.15 0.20" />
       </geometry>
     </collision>
@@ -109,5 +109,5 @@
     <collision>
       <geometry>
-        <box size="0.02 0.02 0.02" />
+        <box size="0.35 0.25 0.15" />
       </geometry>
     </collision>
@@ -126,5 +126,5 @@
     <dynamics damping="0.5"/>
   </joint>
-    <link name="part4_base">
+  <link name="part4_base">
     <visual>
       <origin rpy="0 0 0" xyz="0 0 0"/>
@@ -135,5 +135,5 @@
     <collision>
       <geometry>
-        <box size="0.02 0.02 0.02" />
+        <box size="0.10 0.10 0.10" />
       </geometry>
     </collision>
@@ -161,5 +161,5 @@
     <collision>
       <geometry>
-        <box size="0.02 0.02 0.02" />
+        <mesh filename="package://g500arm5_description/meshes/ARM5E/ARM5E_part4_jaw1.dae"/>
       </geometry>
     </collision>
@@ -187,5 +187,5 @@
     <collision>
       <geometry>
-        <box size="0.02 0.02 0.02" />
+        <mesh filename="package://g500arm5_description/meshes/ARM5E/ARM5E_part4_jaw2.dae"/>
       </geometry>
     </collision>
